File: jupiter-nano/sama5d27-power1.sch (KiCad schematic (older format))
At the start: 50 parts, among them U1 ATSAMA5D27C-LD1G-CU

Commit message: ERC corrections
Parts:
- gave numbers to parts that had none: 1
Changed lines of the file:
@@
 	2350 6000 2350 6100
 $Comp
-L power:GND #PWR?
+L power:GND #PWR0132
 U 1 1 5FC7E204
 P 2350 7550
-F 0 "#PWR?" H 2350 7300 50  0001 C CNN
+F 0 "#PWR0132" H 2350 7300 50  0001 C CNN
 F 1 "GND" H 2355 7377 50  0000 C CNN
 F 2 "" H 2350 7550 50  0001 C CNN
@@
 	7950 3050 7600 3050
 $Comp
-L power:GND #PWR?
+L power:GND #PWR0133
 U 1 1 5FEF0D49
 P 3900 3050
-F 0 "#PWR?" H 3900 2800 50  0001 C CNN
+F 0 "#PWR0133" H 3900 2800 50  0001 C CNN
 F 1 "GND" H 3905 2877 50  0000 C CNN
 F 2 "" H 3900 3050 50  0001 C CNN
@@
 	7100 2150 7100 2200
 $Comp
-L power:GND #PWR?
+L power:GND #PWR0134
 U 1 1 6015BED8
 P 7100 2200
-F 0 "#PWR?" H 7100 1950 50  0001 C CNN
+F 0 "#PWR0134" H 7100 1950 50  0001 C CNN
 F 1 "GND" H 7105 2027 50  0000 C CNN
 F 2 "" H 7100 2200 50  0001 C CNN
@@
 	6100 4650 5750 4650
 $Comp
-L power:GND #PWR?
+L power:GND #PWR0135
 U 1 1 601D850A
 P 4200 5250
-F 0 "#PWR?" H 4200 5000 50  0001 C CNN
+F 0 "#PWR0135" H 4200 5000 50  0001 C CNN
 F 1 "GND" H 4205 5077 50  0000 C CNN
 F 2 "" H 4200 5250 50  0001 C CNN
@@
 	6450 5650 6100 5650
 $Comp
-L power:GND #PWR?
+L power:GND #PWR0136
 U 1 1 601FB1E3
 P 4200 6250
-F 0 "#PWR?" H 4200 6000 50  0001 C CNN
+F 0 "#PWR0136" H 4200 6000 50  0001 C CNN
 F 1 "GND" H 4205 6077 50  0000 C CNN
 F 2 "" H 4200 6250 50  0001 C CNN
@@
 Connection ~ 5000 7500
 $Comp
-L power:GND #PWR?
+L power:GND #PWR0137
 U 1 1 60495110
 P 5000 7550
-F 0 "#PWR?" H 5000 7300 50  0001 C CNN
+F 0 "#PWR0137" H 5000 7300 50  0001 C CNN
 F 1 "GND" H 5005 7377 50  0000 C CNN
 F 2 "" H 5000 7550 50  0001 C CNN
@@
 	3850 6950 3850 7050
 $Comp
-L power:GND #PWR?
+L power:GND #PWR0138
 U 1 1 604B01C3
 P 3850 7050
-F 0 "#PWR?" H 3850 6800 50  0001 C CNN
+F 0 "#PWR0138" H 3850 6800 50  0001 C CNN
 F 1 "GND" H 3855 6877 50  0000 C CNN
 F 2 "" H 3850 7050 50  0001 C CNN
@@
 	7950 4250 7600 4250
 $Comp
-L power:GND #PWR?
+L power:GND #PWR0139
 U 1 1 5F636B7A
 P 3900 4250
-F 0 "#PWR?" H 3900 4000 50  0001 C CNN
+F 0 "#PWR0139" H 3900 4000 50  0001 C CNN
 F 1 "GND" H 3905 4077 50  0000 C CNN
 F 2 "" H 3900 4250 50  0001 C CNN
@@
 	8700 6100 8500 6100
 $Comp
-L power:GND #PWR?
+L power:GND #PWR0140
 U 1 1 5F845541
 P 8500 6250
-F 0 "#PWR?" H 8500 6000 50  0001 C CNN
+F 0 "#PWR0140" H 8500 6000 50  0001 C CNN
 F 1 "GND" H 8505 6077 50  0000 C CNN
 F 2 "" H 8500 6250 50  0001 C CNN
@@
 Text GLabel 3900 3450 0    50   Input ~ 0
 VDDCORE
-$Comp
-L Device:Ferrite_Bead_Small FB?
-U 1 1 5F91D238
-P 4350 3450
-AR Path="/5F395E67/5F91D238" Ref="FB?"  Part="1"
-AR Path="/5FD740BF/5F91D238" Ref="FB?"  Part="1"
-F 0 "FB?" V 4113 3450 50  0000 C CNN
-F 1 "BLM15AG100SH1D" V 4204 3450 50  0000 C CNN
-F 2 "Capacitor_SMD:C_0402_1005Metric" V 4280 3450 50  0001 C CNN
-F 3 "~" H 4350 3450 50  0001 C CNN
-	1    4350 3450
-	0    1    1    0
-$EndComp
 Wire Wire Line
 	4250 3450 3900 3450
@@
 	4900 3150 4900 3200
 $Comp
-L power:GND #PWR?
+L power:GND #PWR0141
 U 1 1 602286E4
 P 4900 3200
-F 0 "#PWR?" H 4900 2950 50  0001 C CNN
+F 0 "#PWR0141" H 4900 2950 50  0001 C CNN
 F 1 "GND" H 4905 3027 50  0000 C CNN
 F 2 "" H 4900 3200 50  0001 C CNN
@@
 	1    0    0    -1
 $EndComp
+$Comp
+L Device:Ferrite_Bead_Small FB6
+U 1 1 5F91D238
+P 4350 3450
+AR Path="/5F395E67/5F91D238" Ref="FB6"  Part="1"
+AR Path="/5FD740BF/5F91D238" Ref="FB?"  Part="1"
+F 0 "FB6" V 4113 3450 50  0000 C CNN
+F 1 "BLM15AG100SH1D" V 4204 3450 50  0000 C CNN
+F 2 "Capacitor_SMD:C_0402_1005Metric" V 4280 3450 50  0001 C CNN
+F 3 "~" H 4350 3450 50  0001 C CNN
+	1    4350 3450
+	0    1    1    0
+$EndComp
 $EndSCHEMATC
