File: jupiter-nano/USB-UART-bridge.sch (KiCad schematic (older format))
At the start: 0 parts

Commit message: WIP, PIO done
Parts:
- added U?: MCP2200-I-MQ, Package_DFN_QFN:QFN-20-1EP_5x5mm_P0.65mm_EP3.35x3.35mm, symbol Interface_USB:MCP2200-I-MQ
Changed lines of the file:
@@
 Comment4 ""
 $EndDescr
+$Comp
+L Interface_USB:MCP2200-I-MQ U?
+U 1 1 5FE73C8E
+P 5400 3100
+F 0 "U?" H 5400 2211 50  0000 C CNN
+F 1 "MCP2200-I-MQ" H 5400 2120 50  0000 C CNN
+F 2 "Package_DFN_QFN:QFN-20-1EP_5x5mm_P0.65mm_EP3.35x3.35mm" H 6500 2300 50  0001 C CNN
+F 3 "http://ww1.microchip.com/downloads/en/DeviceDoc/200022228D.pdf" H 5400 2100 50  0001 C CNN
+	1    5400 3100
+	1    0    0    -1
+$EndComp
 $EndSCHEMATC

Commit message: WIP, USB-UART and JTAG done
- minor clean up and SD Card form factor still left
Parts:
- added C102: 0.1uF, symbol Device:C
- added C110, C111: 16pF 50V, symbol Device:C
- added C?: C, symbol Device:C
- added D101, D102: LED, symbol Device:LED
- added R101, R102: R_Small, symbol Device:R_Small
- added R103: 10K, symbol Device:R_Small
- added R104: 470R 1%, symbol Device:R_Small
- added Y3: NX3225SA-12MHZ-STD-CSR-3, symbol Device:Crystal_GND24
Connections:
- net at U?.1 (RST): now also R104.2
- net USBU_M: now reaches U?.15 (D-)
- net USBU_P: now reaches U?.16 (D+)
- net VDD_3V3: now reaches U?.18 (VDD)
- net VDD_3V3: now also C?.2, D101.2 (A), D102.2 (A), R103.1
- net at U?.19 (OSC1): now also C111.1, Y3.3
- net at U?.2 (GP7/TxLED): now also R102.1
- net at U?.20 (OSC2): now also C110.1, Y3.1
- net at U?.3 (GP6/RxLED): now also R101.1
- net UART1_TX: now reaches U?.7 (TX)
- net UART1_RX: now reaches U?.9 (RX)
- new net: C102.1, R103.2, R104.1
- new net: D101.1 (K), R101.2
- new net: D102.1 (K), R102.2
- new net GND: C102.2, C110.2, C111.2, C?.1, Y3.2, Y3.4
Other:
- moved on the sheet: U?

Commit message: cleanup
Parts:
- added C?: C, symbol Device:C
- C102: renamed from C?; value C -> 0.1uF
Connections:
- net GND: now also U?.17 (VSS)
Changed lines of the file:
@@
 $EndComp
 $Comp
-L Device:C C?
+L Device:C C102
 U 1 1 601C1871
 P 5900 1950
-F 0 "C?" V 5648 1950 50  0000 C CNN
-F 1 "C" V 5739 1950 50  0000 C CNN
+F 0 "C102" V 5648 1950 50  0000 C CNN
+F 1 "0.1uF" V 5739 1950 50  0000 C CNN
 F 2 "" H 5938 1800 50  0001 C CNN
 F 3 "~" H 5900 1950 50  0001 C CNN
@@
 	0    -1   -1   0
 $EndComp
+Wire Wire Line
+	5550 3850 5550 4350
+$Comp
+L power:GND #PWR?
+U 1 1 601F7854
+P 5550 4350
+F 0 "#PWR?" H 5550 4100 50  0001 C CNN
+F 1 "GND" H 5555 4177 50  0000 C CNN
+F 2 "" H 5550 4350 50  0001 C CNN
+F 3 "" H 5550 4350 50  0001 C CNN
+	1    5550 4350
+	1    0    0    -1
+$EndComp
+$Comp
+L Device:C C?
+U 1 1 601F7CAB
+P 4550 4400
+F 0 "C?" V 4298 4400 50  0000 C CNN
+F 1 "C" V 4389 4400 50  0000 C CNN
+F 2 "" H 4588 4250 50  0001 C CNN
+F 3 "~" H 4550 4400 50  0001 C CNN
+	1    4550 4400
+	0    1    1    0
+$EndComp
 $EndSCHEMATC

Commit message: ERC corrections
Parts:
- removed C?: C, symbol Device:C
- gave numbers to parts that had none: 1
Changed lines of the file:
@@
 $EndDescr
 $Comp
-L Interface_USB:MCP2200-I-MQ U?
+L Interface_USB:MCP2200-I-MQ U3
 U 1 1 5FE73C8E
 P 5550 3050
-F 0 "U?" H 5550 2161 50  0000 C CNN
-F 1 "MCP2200-I-MQ" H 5550 2070 50  0000 C CNN
+F 0 "U3" H 4800 3800 50  0000 C CNN
+F 1 "MCP2200-I-MQ" H 6100 3800 50  0000 C CNN
 F 2 "Package_DFN_QFN:QFN-20-1EP_5x5mm_P0.65mm_EP3.35x3.35mm" H 6650 2250 50  0001 C CNN
 F 3 "http://ww1.microchip.com/downloads/en/DeviceDoc/200022228D.pdf" H 5550 2050 50  0001 C CNN
@@
 P 7500 5050
 AR Path="/5F4A5621/601CDF9C" Ref="#PWR?"  Part="1"
-AR Path="/5F395ED8/601CDF9C" Ref="#PWR?"  Part="1"
-F 0 "#PWR?" H 7500 4800 50  0001 C CNN
+AR Path="/5F395ED8/601CDF9C" Ref="#PWR0101"  Part="1"
+F 0 "#PWR0101" H 7500 4800 50  0001 C CNN
 F 1 "GND" H 7505 4877 50  0000 C CNN
 F 2 "" H 7500 5050 50  0001 C CNN
@@
 P 8000 5050
 AR Path="/5F4A5621/601CDFA2" Ref="#PWR?"  Part="1"
-AR Path="/5F395ED8/601CDFA2" Ref="#PWR?"  Part="1"
-F 0 "#PWR?" H 8000 4800 50  0001 C CNN
+AR Path="/5F395ED8/601CDFA2" Ref="#PWR0102"  Part="1"
+F 0 "#PWR0102" H 8000 4800 50  0001 C CNN
 F 1 "GND" H 8005 4877 50  0000 C CNN
 F 2 "" H 8000 5050 50  0001 C CNN
@@
 P 8450 5050
 AR Path="/5F4A5621/601CDFA8" Ref="#PWR?"  Part="1"
-AR Path="/5F395ED8/601CDFA8" Ref="#PWR?"  Part="1"
-F 0 "#PWR?" H 8450 4800 50  0001 C CNN
+AR Path="/5F395ED8/601CDFA8" Ref="#PWR0103"  Part="1"
+F 0 "#PWR0103" H 8450 4800 50  0001 C CNN
 F 1 "GND" H 8455 4877 50  0000 C CNN
 F 2 "" H 8450 5050 50  0001 C CNN
@@
 P 8000 4150
 AR Path="/5F4A5621/601CDFB5" Ref="#PWR?"  Part="1"
-AR Path="/5F395ED8/601CDFB5" Ref="#PWR?"  Part="1"
-F 0 "#PWR?" H 8000 3900 50  0001 C CNN
+AR Path="/5F395ED8/601CDFB5" Ref="#PWR0104"  Part="1"
+F 0 "#PWR0104" H 8000 3900 50  0001 C CNN
 F 1 "GND" H 8005 3977 50  0000 C CNN
 F 2 "" H 8000 4150 50  0001 C CNN
@@
 	2050 3000 2050 3150
 $Comp
-L power:GND #PWR?
+L power:GND #PWR0105
 U 1 1 601E5B72
 P 2050 3150
-F 0 "#PWR?" H 2050 2900 50  0001 C CNN
+F 0 "#PWR0105" H 2050 2900 50  0001 C CNN
 F 1 "GND" H 2055 2977 50  0000 C CNN
 F 2 "" H 2050 3150 50  0001 C CNN
@@
 	6050 1950 6200 1950
 $Comp
-L power:GND #PWR?
+L power:GND #PWR0106
 U 1 1 601F4FCB
 P 6200 1950
-F 0 "#PWR?" H 6200 1700 50  0001 C CNN
+F 0 "#PWR0106" H 6200 1700 50  0001 C CNN
 F 1 "GND" V 6205 1822 50  0000 R CNN
 F 2 "" H 6200 1950 50  0001 C CNN
@@
 	5550 3850 5550 4350
 $Comp
-L power:GND #PWR?
+L power:GND #PWR0107
 U 1 1 601F7854
 P 5550 4350
-F 0 "#PWR?" H 5550 4100 50  0001 C CNN
+F 0 "#PWR0107" H 5550 4100 50  0001 C CNN
 F 1 "GND" H 5555 4177 50  0000 C CNN
 F 2 "" H 5550 4350 50  0001 C CNN
@@
 	1    0    0    -1
 $EndComp
-$Comp
-L Device:C C?
-U 1 1 601F7CAB
-P 4550 4400
-F 0 "C?" V 4298 4400 50  0000 C CNN
-F 1 "C" V 4389 4400 50  0000 C CNN
-F 2 "" H 4588 4250 50  0001 C CNN
-F 3 "~" H 4550 4400 50  0001 C CNN
-	1    4550 4400
-	0    1    1    0
-$EndComp
 $EndSCHEMATC

Commit message: numerous ERC fixes
- still more to go
Parts:
- added C3: 470nF, symbol Device:C
- renumbered C102 to C1, C102 to C2, C110 to C4, C111 to C5, D101 to D1, D102 to D2, R103 to R1, R104 to R2, R101 to R3, R102 to R4, U3 to U2, Y3 to Y1
Connections:
- net GND: now also U2.14 (V_USB), C3.1, C3.2
- no-connect marks 0 -> 8
Other:
- moved on the sheet: C2
Changed lines of the file:
@@
 $EndDescr
 $Comp
-L Interface_USB:MCP2200-I-MQ U3
+L Interface_USB:MCP2200-I-MQ U2
 U 1 1 5FE73C8E
 P 5550 3050
-F 0 "U3" H 4800 3800 50  0000 C CNN
+F 0 "U2" H 4800 3800 50  0000 C CNN
 F 1 "MCP2200-I-MQ" H 6100 3800 50  0000 C CNN
 F 2 "Package_DFN_QFN:QFN-20-1EP_5x5mm_P0.65mm_EP3.35x3.35mm" H 6650 2250 50  0001 C CNN
@@
 USBU_M
 $Comp
-L Device:R_Small R103
+L Device:R_Small R1
 U 1 1 601BFF8A
 P 2050 2000
-F 0 "R103" H 2109 2046 50  0000 L CNN
+F 0 "R1" H 2109 2046 50  0000 L CNN
 F 1 "10K" H 2109 1955 50  0000 L CNN
 F 2 "" H 2050 2000 50  0001 C CNN
@@
 $EndComp
 $Comp
-L Device:R_Small R102
+L Device:R_Small R4
 U 1 1 601C091A
 P 3500 4100
-F 0 "R102" H 3559 4146 50  0000 L CNN
+F 0 "R4" H 3559 4146 50  0000 L CNN
 F 1 "R_Small" H 3559 4055 50  0000 L CNN
 F 2 "" H 3500 4100 50  0001 C CNN
@@
 $EndComp
 $Comp
-L Device:C C102
+L Device:C C1
 U 1 1 601C0F94
 P 2050 2850
-F 0 "C102" H 2165 2896 50  0000 L CNN
+F 0 "C1" H 2165 2896 50  0000 L CNN
 F 1 "0.1uF" H 2165 2805 50  0000 L CNN
 F 2 "" H 2088 2700 50  0001 C CNN
@@
 $EndComp
 $Comp
-L Device:C C102
+L Device:C C2
 U 1 1 601C1871
-P 5900 1950
-F 0 "C102" V 5648 1950 50  0000 C CNN
-F 1 "0.1uF" V 5739 1950 50  0000 C CNN
-F 2 "" H 5938 1800 50  0001 C CNN
-F 3 "~" H 5900 1950 50  0001 C CNN
-	1    5900 1950
-	0    1    1    0
+P 5000 1950
+F 0 "C2" V 4748 1950 50  0000 C CNN
+F 1 "0.1uF" V 4839 1950 50  0000 C CNN
+F 2 "" H 5038 1800 50  0001 C CNN
+F 3 "~" H 5000 1950 50  0001 C CNN
+	1    5000 1950
+	0    -1   -1   0
 $EndComp
 $Comp
@@
 P 8450 4750
 AR Path="/5F4A5621/601CDF93" Ref="C?"  Part="1"
-AR Path="/5F395ED8/601CDF93" Ref="C111"  Part="1"
-F 0 "C111" H 8565 4796 50  0000 L CNN
+AR Path="/5F395ED8/601CDF93" Ref="C5"  Part="1"
+F 0 "C5" H 8565 4796 50  0000 L CNN
 F 1 "16pF 50V" H 8565 4705 50  0000 L CNN
 F 2 "" H 8488 4600 50  0001 C CNN
@@
 P 7500 5050
 AR Path="/5F4A5621/601CDF9C" Ref="#PWR?"  Part="1"
-AR Path="/5F395ED8/601CDF9C" Ref="#PWR0101"  Part="1"
-F 0 "#PWR0101" H 7500 4800 50  0001 C CNN
+AR Path="/5F395ED8/601CDF9C" Ref="#PWR05"  Part="1"
+F 0 "#PWR05" H 7500 4800 50  0001 C CNN
 F 1 "GND" H 7505 4877 50  0000 C CNN
 F 2 "" H 7500 5050 50  0001 C CNN
@@
 P 8000 5050
 AR Path="/5F4A5621/601CDFA2" Ref="#PWR?"  Part="1"
-AR Path="/5F395ED8/601CDFA2" Ref="#PWR0102"  Part="1"
-F 0 "#PWR0102" H 8000 4800 50  0001 C CNN
+AR Path="/5F395ED8/601CDFA2" Ref="#PWR07"  Part="1"
+F 0 "#PWR07" H 8000 4800 50  0001 C CNN
 F 1 "GND" H 8005 4877 50  0000 C CNN
 F 2 "" H 8000 5050 50  0001 C CNN
@@
 P 8450 5050
 AR Path="/5F4A5621/601CDFA8" Ref="#PWR?"  Part="1"
-AR Path="/5F395ED8/601CDFA8" Ref="#PWR0103"  Part="1"
-F 0 "#PWR0103" H 8450 4800 50  0001 C CNN
+AR Path="/5F395ED8/601CDFA8" Ref="#PWR08"  Part="1"
+F 0 "#PWR08" H 8450 4800 50  0001 C CNN
 F 1 "GND" H 8455 4877 50  0000 C CNN
 F 2 "" H 8450 5050 50  0001 C CNN
@@
 P 8000 4150
 AR Path="/5F4A5621/601CDFB5" Ref="#PWR?"  Part="1"
-AR Path="/5F395ED8/601CDFB5" Ref="#PWR0104"  Part="1"
-F 0 "#PWR0104" H 8000 3900 50  0001 C CNN
+AR Path="/5F395ED8/601CDFB5" Ref="#PWR06"  Part="1"
+F 0 "#PWR06" H 8000 3900 50  0001 C CNN
 F 1 "GND" H 8005 3977 50  0000 C CNN
 F 2 "" H 8000 4150 50  0001 C CNN
@@
 P 8000 4500
 AR Path="/5F4A5621/601CDFBE" Ref="Y?"  Part="1"
-AR Path="/5F395ED8/601CDFBE" Ref="Y3"  Part="1"
-F 0 "Y3" H 7750 4600 50  0000 L CNN
+AR Path="/5F395ED8/601CDFBE" Ref="Y1"  Part="1"
+F 0 "Y1" H 7750 4600 50  0000 L CNN
 F 1 "NX3225SA-12MHZ-STD-CSR-3 " H 8200 4600 50  0000 L CNN
 F 2 "" H 8000 4500 50  0001 C CNN
@@
 	2050 3000 2050 3150
 $Comp
-L power:GND #PWR0105
+L power:GND #PWR01
 U 1 1 601E5B72
 P 2050 3150
-F 0 "#PWR0105" H 2050 2900 50  0001 C CNN
+F 0 "#PWR01" H 2050 2900 50  0001 C CNN
 F 1 "GND" H 2055 2977 50  0000 C CNN
 F 2 "" H 2050 3150 50  0001 C CNN
@@
 	4650 2450 2650 2450
 $Comp
-L Device:R_Small R104
+L Device:R_Small R2
 U 1 1 601BF9F4
 P 2550 2450
-F 0 "R104" V 2746 2450 50  0000 C CNN
+F 0 "R2" V 2746 2450 50  0000 C CNN
 F 1 "470R 1%" V 2655 2450 50  0000 C CNN
 F 2 "" H 2550 2450 50  0001 C CNN
@@
 $EndComp
 $Comp
-L Device:LED D102
+L Device:LED D2
 U 1 1 601ED675
 P 3500 4500
-F 0 "D102" V 3447 4580 50  0000 L CNN
+F 0 "D2" V 3447 4580 50  0000 L CNN
 F 1 "LED" V 3538 4580 50  0000 L CNN
 F 2 "" H 3500 4500 50  0001 C CNN
@@
 $EndComp
 $Comp
-L Device:LED D101
+L Device:LED D1
 U 1 1 601EEDED
 P 2950 4500
-F 0 "D101" V 2897 4580 50  0000 L CNN
+F 0 "D1" V 2897 4580 50  0000 L CNN
 F 1 "LED" V 2988 4580 50  0000 L CNN
 F 2 "" H 2950 4500 50  0001 C CNN
@@
 P 7500 4750
 AR Path="/5F4A5621/601CDF8D" Ref="C?"  Part="1"
-AR Path="/5F395ED8/601CDF8D" Ref="C110"  Part="1"
-F 0 "C110" H 7615 4796 50  0000 L CNN
+AR Path="/5F395ED8/601CDF8D" Ref="C4"  Part="1"
+F 0 "C4" H 7615 4796 50  0000 L CNN
 F 1 "16pF 50V" H 7615 4705 50  0000 L CNN
 F 2 "" H 7538 4600 50  0001 C CNN
@@
 $EndComp
 $Comp
-L Device:R_Small R101
+L Device:R_Small R3
 U 1 1 601C05B7
 P 2950 4100
-F 0 "R101" H 3009 4146 50  0000 L CNN
+F 0 "R3" H 3009 4146 50  0000 L CNN
 F 1 "R_Small" H 3009 4055 50  0000 L CNN
 F 2 "" H 2950 4100 50  0001 C CNN
@@
 VDD_3V3
 Wire Wire Line
-	5750 1950 5450 1950
+	5150 1950 5450 1950
 Connection ~ 5450 1950
 Wire Wire Line
 	5450 1950 5450 2250
 Wire Wire Line
-	6050 1950 6200 1950
-$Comp
-L power:GND #PWR0106
+	4850 1950 4700 1950
+$Comp
+L power:GND #PWR02
 U 1 1 601F4FCB
-P 6200 1950
-F 0 "#PWR0106" H 6200 1700 50  0001 C CNN
-F 1 "GND" V 6205 1822 50  0000 R CNN
-F 2 "" H 6200 1950 50  0001 C CNN
-F 3 "" H 6200 1950 50  0001 C CNN
-	1    6200 1950
-	0    -1   -1   0
-$EndComp
-Wire Wire Line
-	5550 3850 5550 4350
-$Comp
-L power:GND #PWR0107
+P 4700 1950
+F 0 "#PWR02" H 4700 1700 50  0001 C CNN
+F 1 "GND" V 4705 1822 50  0000 R CNN
+F 2 "" H 4700 1950 50  0001 C CNN
+F 3 "" H 4700 1950 50  0001 C CNN
+	1    4700 1950
+	0    1    1    0
+$EndComp
+Wire Wire Line
+	5550 3850 5550 4050
+$Comp
+L power:GND #PWR03
 U 1 1 601F7854
 P 5550 4350
-F 0 "#PWR0107" H 5550 4100 50  0001 C CNN
+F 0 "#PWR03" H 5550 4100 50  0001 C CNN
 F 1 "GND" H 5555 4177 50  0000 C CNN
 F 2 "" H 5550 4350 50  0001 C CNN
@@
 	1    0    0    -1
 $EndComp
+NoConn ~ 4650 2850
+NoConn ~ 4650 2950
+NoConn ~ 4650 3050
+NoConn ~ 4650 3150
+NoConn ~ 4650 3250
+NoConn ~ 4650 3350
+NoConn ~ 4650 3450
+$Comp
+L power:GND #PWR04
+U 1 1 60422D0E
+P 6100 1500
+F 0 "#PWR04" H 6100 1250 50  0001 C CNN
+F 1 "GND" H 6105 1327 50  0000 C CNN
+F 2 "" H 6100 1500 50  0001 C CNN
+F 3 "" H 6100 1500 50  0001 C CNN
+	1    6100 1500
+	-1   0    0    1
+$EndComp
+Wire Wire Line
+	6100 1500 6100 1650
+$Comp
+L Device:C C3
+U 1 1 60421769
+P 6100 1800
+F 0 "C3" H 6215 1846 50  0000 L CNN
+F 1 "470nF" H 6215 1755 50  0000 L CNN
+F 2 "" H 6138 1650 50  0001 C CNN
+F 3 "~" H 6100 1800 50  0001 C CNN
+	1    6100 1800
+	1    0    0    -1
+$EndComp
+Wire Wire Line
+	6100 1950 5650 1950
+Wire Wire Line
+	5650 1950 5650 2250
+NoConn ~ 4650 2750
+Wire Wire Line
+	5550 4050 6700 4050
+Wire Wire Line
+	6700 4050 6700 1950
+Wire Wire Line
+	6700 1950 6100 1950
+Connection ~ 5550 4050
+Wire Wire Line
+	5550 4050 5550 4350
+Connection ~ 6100 1950
 $EndSCHEMATC
