File: jupiter-nano/sama5d27-clock.sch (KiCad schematic (older format))
At the start: 14 parts, among them U1 ATSAMA5D27C-LD1G-CU, Y2 NX3225SA-12MHZ-STD-CSR-3, Y3 NX2012SA-32.768KHZ-EXS00A-MU0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

Commit message: added at24csw080 I2C EEPROM UUID chip
Parts:
- added R201: 100K DNP, symbol Device:R_Small
- renumbered R14 to R17, R15 to R18, R16 to R19, R17 to R20, R18 to R21
Connections:
- net at U1.T3 (JTAGSEL): now also R201.1
- new net VDDBU: R201.2
- no-connect marks 4 -> 3
Other:
- note added: "Place this resistor to disable JTAG debugging."
Changed lines of the file:
@@
 $EndComp
 $Comp
-L Device:R_Small R14
+L Device:R_Small R17
 U 1 1 5FB9019B
 P 4150 2750
-F 0 "R14" V 4200 2600 50  0000 C CNN
+F 0 "R17" V 4200 2600 50  0000 C CNN
 F 1 "100R 1%" V 4200 3000 50  0000 C CNN
 F 2 "" H 4150 2750 50  0001 C CNN
@@
 $EndComp
 $Comp
-L Device:R_Small R16
+L Device:R_Small R19
 U 1 1 5FB90BC4
 P 4200 3200
-F 0 "R16" V 4250 3050 50  0000 C CNN
+F 0 "R19" V 4250 3050 50  0000 C CNN
 F 1 "10K" V 4250 3450 50  0000 C CNN
 F 2 "" H 4200 3200 50  0001 C CNN
@@
 $EndComp
 $Comp
-L Device:R_Small R17
+L Device:R_Small R20
 U 1 1 5FB913F4
 P 7350 2700
-F 0 "R17" V 7250 2700 50  0000 C CNN
+F 0 "R20" V 7250 2700 50  0000 C CNN
 F 1 "100R 1%" V 7450 2750 50  0000 C CNN
 F 2 "" H 7350 2700 50  0001 C CNN
@@
 $EndComp
 $Comp
-L Device:R_Small R15
+L Device:R_Small R18
 U 1 1 5FB91AFA
 P 4150 3050
-F 0 "R15" V 4200 2900 50  0000 C CNN
+F 0 "R18" V 4200 2900 50  0000 C CNN
 F 1 "100R 1%" V 4200 3300 50  0000 C CNN
 F 2 "" H 4150 3050 50  0001 C CNN
@@
 	3850 3050 4050 3050
 $Comp
-L power:GND #PWR031
+L power:GND #PWR032
 U 1 1 5FBB7C84
 P 3850 3050
-F 0 "#PWR031" H 3850 2800 50  0001 C CNN
+F 0 "#PWR032" H 3850 2800 50  0001 C CNN
 F 1 "GND" V 3855 2922 50  0000 R CNN
 F 2 "" H 3850 3050 50  0001 C CNN
@@
 Connection ~ 8400 3650
 $Comp
-L power:GND #PWR032
+L power:GND #PWR033
 U 1 1 5FBD26A3
 P 8400 4050
-F 0 "#PWR032" H 8400 3800 50  0001 C CNN
+F 0 "#PWR033" H 8400 3800 50  0001 C CNN
 F 1 "GND" H 8405 3877 50  0000 C CNN
 F 2 "" H 8400 4050 50  0001 C CNN
@@
 	2250 4050 2250 4200
 $Comp
-L power:GND #PWR025
+L power:GND #PWR026
 U 1 1 5FE58F04
 P 1300 4200
-F 0 "#PWR025" H 1300 3950 50  0001 C CNN
+F 0 "#PWR026" H 1300 3950 50  0001 C CNN
 F 1 "GND" H 1305 4027 50  0000 C CNN
 F 2 "" H 1300 4200 50  0001 C CNN
@@
 $EndComp
 $Comp
-L power:GND #PWR027
+L power:GND #PWR028
 U 1 1 5FE592EB
 P 1800 4200
-F 0 "#PWR027" H 1800 3950 50  0001 C CNN
+F 0 "#PWR028" H 1800 3950 50  0001 C CNN
 F 1 "GND" H 1805 4027 50  0000 C CNN
 F 2 "" H 1800 4200 50  0001 C CNN
@@
 $EndComp
 $Comp
-L power:GND #PWR028
+L power:GND #PWR029
 U 1 1 5FE59993
 P 2250 4200
-F 0 "#PWR028" H 2250 3950 50  0001 C CNN
+F 0 "#PWR029" H 2250 3950 50  0001 C CNN
 F 1 "GND" H 2255 4027 50  0000 C CNN
 F 2 "" H 2250 4200 50  0001 C CNN
@@
 	1800 3450 1800 3300
 $Comp
-L power:GND #PWR026
+L power:GND #PWR027
 U 1 1 5FE62514
 P 1800 3300
-F 0 "#PWR026" H 1800 3050 50  0001 C CNN
+F 0 "#PWR027" H 1800 3050 50  0001 C CNN
 F 1 "GND" H 1805 3127 50  0000 C CNN
 F 2 "" H 1800 3300 50  0001 C CNN
@@
 Connection ~ 3800 4800
 $Comp
-L power:GND #PWR029
+L power:GND #PWR030
 U 1 1 5FE6D6B8
 P 2850 5350
-F 0 "#PWR029" H 2850 5100 50  0001 C CNN
+F 0 "#PWR030" H 2850 5100 50  0001 C CNN
 F 1 "GND" H 2855 5177 50  0000 C CNN
 F 2 "" H 2850 5350 50  0001 C CNN
@@
 $EndComp
 $Comp
-L power:GND #PWR030
+L power:GND #PWR031
 U 1 1 5FE6DCB8
 P 3800 5350
-F 0 "#PWR030" H 3800 5100 50  0001 C CNN
+F 0 "#PWR031" H 3800 5100 50  0001 C CNN
 F 1 "GND" H 3805 5177 50  0000 C CNN
 F 2 "" H 3800 5350 50  0001 C CNN
@@
 	8400 3950 8400 4050
 $Comp
-L Device:R_Small R18
+L Device:R_Small R21
 U 1 1 5FB8F66D
 P 8400 3300
-F 0 "R18" H 8459 3346 50  0000 L CNN
+F 0 "R21" H 8459 3346 50  0000 L CNN
 F 1 "5.6K" H 8459 3255 50  0000 L CNN
 F 2 "" H 8400 3300 50  0001 C CNN
@@
 NoConn ~ 4450 2250
 NoConn ~ 4450 2350
-NoConn ~ 4450 2600
 NoConn ~ 4450 2900
+Text GLabel 3800 2600 0    50   Input ~ 0
+VDDBU
+$Comp
+L Device:R_Small R201
+U 1 1 5F6AD118
+P 4150 2600
+F 0 "R201" V 4200 2400 50  0000 C CNN
+F 1 "100K DNP" V 4200 2900 50  0000 C CNN
+F 2 "" H 4150 2600 50  0001 C CNN
+F 3 "~" H 4150 2600 50  0001 C CNN
+	1    4150 2600
+	0    1    1    0
+$EndComp
+Wire Wire Line
+	3800 2600 4050 2600
+Wire Wire Line
+	4250 2600 4450 2600
+Text Notes 2950 2500 0    50   ~ 0
+Place this resistor to disable JTAG debugging.
 $EndSCHEMATC
