File: jupiter-nano/sama5d27-power2.sch (KiCad schematic (older format))
At the start: 1 part, among them U1 ATSAMA5D27C-LD1G-CU

Commit message: WIP, power done
Parts:
- added C39, C?: 4.7uF, symbol Device:C
- added C44, C52, C56, C?: 0.1uF, symbol Device:C
- added FB7: BLM15AG100SH1D, Capacitor_SMD:C_0402_1005Metric, symbol Device:Ferrite_Bead_Small
- added L6: MLZ1608M100L, symbol pspice:INDUCTOR
- added R17: 2.2R, symbol Device:R_Small
Connections:
- net labels added: VDDCORE, VDDOSC, VDD_UTIMII
- net labels removed: VDD_UTMI
- wire segments 95 -> 129

Commit message: WIP clocking done
Parts:
- gave numbers to parts that had none: 2
Other:
- moved on the sheet: U1H

Commit message: numerous ERC fixes
- still more to go
Parts:
- renumbered C52 to C78, C56 to C79, C41 to C80, C39 to C81, C45 to C82, C44 to C83, FB7 to FB3, L6 to L4, R17 to R40
Changed lines of the file:
@@
 	4100 3800 4350 3800
 $Comp
-L power:GND #PWR0164
+L power:GND #PWR065
 U 1 1 5FC8B21F
 P 4100 6050
-F 0 "#PWR0164" H 4100 5800 50  0001 C CNN
+F 0 "#PWR065" H 4100 5800 50  0001 C CNN
 F 1 "GND" H 4105 5877 50  0000 C CNN
 F 2 "" H 4100 6050 50  0001 C CNN
@@
 P 7400 3500
 AR Path="/5F395E67/5FAB62AA" Ref="C?"  Part="1"
-AR Path="/5FB0A4D9/5FAB62AA" Ref="C56"  Part="1"
-F 0 "C56" H 7400 3600 50  0000 L CNN
+AR Path="/5FB0A4D9/5FAB62AA" Ref="C79"  Part="1"
+F 0 "C79" H 7400 3600 50  0000 L CNN
 F 1 "0.1uF" H 7400 3400 50  0000 L CNN
 F 2 "" H 7438 3350 50  0001 C CNN
@@
 P 7050 3500
 AR Path="/5F395E67/5FAB62B0" Ref="C?"  Part="1"
-AR Path="/5FB0A4D9/5FAB62B0" Ref="C52"  Part="1"
-F 0 "C52" H 7050 3600 50  0000 L CNN
+AR Path="/5FB0A4D9/5FAB62B0" Ref="C78"  Part="1"
+F 0 "C78" H 7050 3600 50  0000 L CNN
 F 1 "0.1uF" H 7050 3400 50  0000 L CNN
 F 2 "" H 7088 3350 50  0001 C CNN
@@
 P 7250 3950
 AR Path="/5F395E67/5FAB62BD" Ref="#PWR?"  Part="1"
-AR Path="/5FB0A4D9/5FAB62BD" Ref="#PWR0165"  Part="1"
-F 0 "#PWR0165" H 7250 3700 50  0001 C CNN
+AR Path="/5FB0A4D9/5FAB62BD" Ref="#PWR066"  Part="1"
+F 0 "#PWR066" H 7250 3700 50  0001 C CNN
 F 1 "GND" H 7255 3777 50  0000 C CNN
 F 2 "" H 7250 3950 50  0001 C CNN
@@
 AR Path="/5F395E67/5FAFAB51" Ref="FB?"  Part="1"
 AR Path="/5FD740BF/5FAFAB51" Ref="FB?"  Part="1"
-AR Path="/5FB0A4D9/5FAFAB51" Ref="FB7"  Part="1"
-F 0 "FB7" V 9413 3800 50  0000 C CNN
+AR Path="/5FB0A4D9/5FAFAB51" Ref="FB3"  Part="1"
+F 0 "FB3" V 9413 3800 50  0000 C CNN
 F 1 "BLM15AG100SH1D" V 9504 3800 50  0000 C CNN
 F 2 "Capacitor_SMD:C_0402_1005Metric" V 9580 3800 50  0001 C CNN
@@
 P 8700 4150
 AR Path="/5F395E67/5FB1650F" Ref="C?"  Part="1"
-AR Path="/5FB0A4D9/5FB1650F" Ref="C39"  Part="1"
-F 0 "C39" H 8700 4250 50  0000 L CNN
+AR Path="/5FB0A4D9/5FB1650F" Ref="C81"  Part="1"
+F 0 "C81" H 8700 4250 50  0000 L CNN
 F 1 "4.7uF" H 8700 4050 50  0000 L CNN
 F 2 "" H 8738 4000 50  0001 C CNN
@@
 P 9100 4150
 AR Path="/5F395E67/5FB212DA" Ref="C?"  Part="1"
-AR Path="/5FB0A4D9/5FB212DA" Ref="C44"  Part="1"
-F 0 "C44" H 9100 4250 50  0000 L CNN
+AR Path="/5FB0A4D9/5FB212DA" Ref="C83"  Part="1"
+F 0 "C83" H 9100 4250 50  0000 L CNN
 F 1 "0.1uF" H 9100 4050 50  0000 L CNN
 F 2 "" H 9138 4000 50  0001 C CNN
@@
 P 8900 4550
 AR Path="/5F395E67/5FB2565C" Ref="#PWR?"  Part="1"
-AR Path="/5FB0A4D9/5FB2565C" Ref="#PWR0166"  Part="1"
-F 0 "#PWR0166" H 8900 4300 50  0001 C CNN
+AR Path="/5FB0A4D9/5FB2565C" Ref="#PWR068"  Part="1"
+F 0 "#PWR068" H 8900 4300 50  0001 C CNN
 F 1 "GND" H 8905 4377 50  0000 C CNN
 F 2 "" H 8900 4550 50  0001 C CNN
@@
 P 8500 2400
 AR Path="/5F395E67/5FB30433" Ref="C?"  Part="1"
-AR Path="/5FB0A4D9/5FB30433" Ref="C41"  Part="1"
-F 0 "C41" H 8500 2500 50  0000 L CNN
+AR Path="/5FB0A4D9/5FB30433" Ref="C80"  Part="1"
+F 0 "C80" H 8500 2500 50  0000 L CNN
 F 1 "4.7uF" H 8500 2300 50  0000 L CNN
 F 2 "" H 8538 2250 50  0001 C CNN
@@
 P 8900 2400
 AR Path="/5F395E67/5FB3043D" Ref="C?"  Part="1"
-AR Path="/5FB0A4D9/5FB3043D" Ref="C45"  Part="1"
-F 0 "C45" H 8900 2500 50  0000 L CNN
+AR Path="/5FB0A4D9/5FB3043D" Ref="C82"  Part="1"
+F 0 "C82" H 8900 2500 50  0000 L CNN
 F 1 "0.1uF" H 8900 2300 50  0000 L CNN
 F 2 "" H 8938 2250 50  0001 C CNN
@@
 P 8700 2800
 AR Path="/5F395E67/5FB3044A" Ref="#PWR?"  Part="1"
-AR Path="/5FB0A4D9/5FB3044A" Ref="#PWR0167"  Part="1"
-F 0 "#PWR0167" H 8700 2550 50  0001 C CNN
+AR Path="/5FB0A4D9/5FB3044A" Ref="#PWR067"  Part="1"
+F 0 "#PWR067" H 8700 2550 50  0001 C CNN
 F 1 "GND" H 8705 2627 50  0000 C CNN
 F 2 "" H 8700 2800 50  0001 C CNN
@@
 P 9500 2050
 AR Path="/5F549DCF/5FB6E3C5" Ref="L?"  Part="1"
-AR Path="/5FB0A4D9/5FB6E3C5" Ref="L6"  Part="1"
-F 0 "L6" H 9500 2200 50  0000 C CNN
+AR Path="/5FB0A4D9/5FB6E3C5" Ref="L4"  Part="1"
+F 0 "L4" H 9500 2200 50  0000 C CNN
 F 1 "MLZ1608M100L" H 9500 2000 50  0000 C CNN
 F 2 "" H 9500 2050 50  0001 C CNN
@@
 VDDCORE
 $Comp
-L Device:R_Small R17
+L Device:R_Small R40
 U 1 1 5FB72AC9
 P 10100 2050
-F 0 "R17" V 9904 2050 50  0000 C CNN
+F 0 "R40" V 9904 2050 50  0000 C CNN
 F 1 "2.2R" V 9995 2050 50  0000 C CNN
 F 2 "" H 10100 2050 50  0001 C CNN

Commit message: added at24csw080 I2C EEPROM UUID chip
Parts:
- renumbered R40 to R43
Connections:
- net VDDIOP2 is gone; now on net VDDIOP1: U1.A8 (VDDIOP2)
- net VDD_3V3 is gone; now on net VDDIOP1: C78.1, C79.1, U1.G3 (VDDISC), U1.T7 (VDDSDMMC)
- net VDD_UTIMII renamed VDDUTMII
Other:
- note added: "Power Links"
Changed lines of the file:
@@
 	4100 3800 4350 3800
 $Comp
-L power:GND #PWR065
+L power:GND #PWR066
 U 1 1 5FC8B21F
 P 4100 6050
-F 0 "#PWR065" H 4100 5800 50  0001 C CNN
+F 0 "#PWR066" H 4100 5800 50  0001 C CNN
 F 1 "GND" H 4105 5877 50  0000 C CNN
 F 2 "" H 4100 6050 50  0001 C CNN
@@
 P 7250 3950
 AR Path="/5F395E67/5FAB62BD" Ref="#PWR?"  Part="1"
-AR Path="/5FB0A4D9/5FAB62BD" Ref="#PWR066"  Part="1"
-F 0 "#PWR066" H 7250 3700 50  0001 C CNN
+AR Path="/5FB0A4D9/5FAB62BD" Ref="#PWR067"  Part="1"
+F 0 "#PWR067" H 7250 3700 50  0001 C CNN
 F 1 "GND" H 7255 3777 50  0000 C CNN
 F 2 "" H 7250 3950 50  0001 C CNN
@@
 	6950 2550 7500 2550
 Text GLabel 7500 2550 2    50   Input ~ 0
-VDD_UTIMII
+VDDUTMII
 Wire Wire Line
 	7050 2250 7050 3350
@@
 P 8900 4550
 AR Path="/5F395E67/5FB2565C" Ref="#PWR?"  Part="1"
-AR Path="/5FB0A4D9/5FB2565C" Ref="#PWR068"  Part="1"
-F 0 "#PWR068" H 8900 4300 50  0001 C CNN
+AR Path="/5FB0A4D9/5FB2565C" Ref="#PWR069"  Part="1"
+F 0 "#PWR069" H 8900 4300 50  0001 C CNN
 F 1 "GND" H 8905 4377 50  0000 C CNN
 F 2 "" H 8900 4550 50  0001 C CNN
@@
 P 8700 2800
 AR Path="/5F395E67/5FB3044A" Ref="#PWR?"  Part="1"
-AR Path="/5FB0A4D9/5FB3044A" Ref="#PWR067"  Part="1"
-F 0 "#PWR067" H 8700 2550 50  0001 C CNN
+AR Path="/5FB0A4D9/5FB3044A" Ref="#PWR068"  Part="1"
+F 0 "#PWR068" H 8700 2550 50  0001 C CNN
 F 1 "GND" H 8705 2627 50  0000 C CNN
 F 2 "" H 8700 2800 50  0001 C CNN
@@
 VDDCORE
 $Comp
-L Device:R_Small R40
+L Device:R_Small R43
 U 1 1 5FB72AC9
 P 10100 2050
-F 0 "R40" V 9904 2050 50  0000 C CNN
+F 0 "R43" V 9904 2050 50  0000 C CNN
 F 1 "2.2R" V 9995 2050 50  0000 C CNN
 F 2 "" H 10100 2050 50  0001 C CNN
@@
 Connection ~ 4100 3700
 Connection ~ 4100 3800
+Text GLabel 1250 1150 0    50   Input ~ 0
+VDD_3V3
+Text GLabel 1800 1150 2    50   Input ~ 0
+VDDIOP1
+Text Notes 1900 850  2    79   ~ 16
+Power Links
+Wire Wire Line
+	1250 1150 1800 1150
+Text GLabel 1250 1400 0    50   Input ~ 0
+VDD_3V3
+Text GLabel 1800 1400 2    50   Input ~ 0
+VDDIOP2
+Wire Wire Line
+	1250 1400 1800 1400
 $EndSCHEMATC
